File: hardware/electronics/KELPIE_INPUT_PCB.brd (EAGLE design)
At the start: 101.6 x 57.1 mm, 27 parts, among them J1 30_PIN_CONNECTOR_MALE

Commit message: upper PCB revisions
Parts:
- D1: device sirin-clone-library:CHIPLED_0805 -> sirin-clone-library:LEDRD254W60D400H525B
- J1: value 30_PIN_CONNECTOR_MALE -> 30_PIN_CONNECTOR_MALEFLEX_CONNECTOR; device sirin-clone-library:MOLEX_30PINCONNECTOR_2MM -> sirin-clone-library:SLW30S
- moved R5 12.0 mm to (21.0, 53.0), turned to 0 degrees
- moved J1 0.95 mm to (81.3, 53.0), flipped to the bottom, turned to 180 degrees
- moved D1 0.63 mm to (9.53, 53.3)
Connections:
- net 3.3V: now also J1.14, J1.15; no longer J1.P$14, J1.P$15
- net AGND: now also J1.29, J1.30; no longer J1.P$29, J1.P$30
- net GND: now also D1.2, J1.13; no longer D1.C, J1.P$13
- net N$6: now also D1.1; no longer D1.A
- net PIN15/KNOB1(VOL): now also J1.24; no longer J1.P$24
- net PIN16/KNOB2: now also J1.28; no longer J1.P$28
- net PIN17/KNOB3: now also J1.27; no longer J1.P$27
- net PIN2/SW1: now also J1.19; no longer J1.P$19
- net PIN20/KNOB4: now also J1.3; no longer J1.P$3
- net PIN21/KNOB5: now also J1.4; no longer J1.P$4
- net PIN24/LED1: now also J1.16; no longer J1.P$16
- net PIN25/LED2: now also J1.25; no longer J1.P$25
- net PIN26/KNOB6: now also J1.8; no longer J1.P$8
- net PIN27/KNOB7: now also J1.22; no longer J1.P$22
- net PIN28/KNOB8: now also J1.23; no longer J1.P$23
- net PIN29/KNOB9: now also J1.21; no longer J1.P$21
- net PIN3/SW2: now also J1.17; no longer J1.P$17
- net PIN30/KNOB10: now also J1.20; no longer J1.P$20
- net PIN31/KNOB11: now also J1.7; no longer J1.P$7
- net PIN32/LED3: now also J1.26; no longer J1.P$26
- net PIN33/LED4: now also J1.1; no longer J1.P$1
- net PIN4/SW3: now also J1.18; no longer J1.P$18
- net PIN5/SW4: now also J1.5; no longer J1.P$5
- net PIN8/MIDILED: now also J1.2; no longer J1.P$2
- net PINA10/KNOB12: now also J1.10; no longer J1.P$10
- net PINA11/KNOB13: now also J1.9; no longer J1.P$9
- net PINA12/KNOB14: now also J1.11; no longer J1.P$11
- net PINA13/KNOB15: now also J1.12; no longer J1.P$12
- net PINA14/KNOB16: now also J1.6; no longer J1.P$6
Routing:
- net PIN8/MIDILED: track 66.1 -> 49.2 mm, vias 9 -> 6
- net PIN5/SW4: track 53.3 -> 59.0 mm, vias 3 -> 1
- net PIN33/LED4: track 63.2 -> 68.3 mm, vias 1 -> 2
- net PIN21/KNOB5: track 35.3 -> 39.5 mm
- net PIN32/LED3: track 93.3 -> 89.8 mm, vias 5 -> 3
- net PIN20/KNOB4: track 51.6 -> 54.9 mm
- net PIN27/KNOB7: track 57.1 -> 60.3 mm
- net PINA13/KNOB15: track 53.1 -> 50.2 mm, vias 5 -> 4
- net PIN28/KNOB8: track 41.1 -> 44.0 mm
- net PIN15/KNOB1(VOL): track 25.2 -> 28.0 mm
- net GND: track 239.3 -> 236.5 mm
- net PIN25/LED2: track 84.8 -> 87.5 mm
- net PIN24/LED1: track 87.6 -> 90.4 mm
- net PIN30/KNOB10: track 49.9 -> 52.7 mm
- net PIN2/SW1: track 89.1 -> 91.8 mm
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Other:
- outline, holes or cut-outs redrawn
