File: hardware/electronics/KELPIE_LOGIC_PCB.sch (EAGLE design)
At the start: 55 parts, among them J1 PJ-002A, J3 30_PIN_CONNECTOR_MALEFLEX_CON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, J5 SWITCHCRAFT_PHONEJACK, J6 SWD_CONNECTOR, T2 MCP1825S, U4 SGTL5000_32QFN, U5 23LC1024

Commit message: board rev 2 done, sent to seeed for manufacture
Parts:
- added U$2: TEST_POINT, sirin-clone-library:TEST_POINT
Connections:
- net VUSB_IN: now also U$2.P$1
Changed lines of the file:
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@@
 <?xml version="1.0" encoding="utf-8"?>
 <!DOCTYPE eagle SYSTEM "eagle.dtd">
-<eagle version="9.4.2">
+<eagle version="9.3.1">
 <drawing>
 <settings>
@@
 <part name="GND1" library="sirin-clone-library" library_urn="urn:adsk.eagle:library:9336050" deviceset="GND" device=""/>
 <part name="GND2" library="sirin-clone-library" library_urn="urn:adsk.eagle:library:9336050" deviceset="GND" device=""/>
-<part name="J3" library="sirin-clone-library" library_urn="urn:adsk.eagle:library:9336050" deviceset="30_PIN_CONNECTOR_MALE" device="FLEX_CONNECTOR" package3d_urn="urn:adsk.eagle:package:12919137/6" value="30_PIN_CONNECTOR_MALEFLEX_CONNECTOR"/>
+<part name="J3" library="sirin-clone-library" library_urn="urn:adsk.eagle:library:9336050" deviceset="30_PIN_CONNECTOR_MALE" device="FLEX_CONNECTOR" package3d_urn="urn:adsk.eagle:package:12919137/7" value="30_PIN_CONNECTOR_MALEFLEX_CONNECTOR"/>
 <part name="GND3" library="sirin-clone-library" library_urn="urn:adsk.eagle:library:9336050" deviceset="GND" device=""/>
 <part name="K3" library="moon-germs-v1_main" library_urn="urn:adsk.eagle:library:8442267" deviceset="MK20DX256VLH7" device="" package3d_urn="urn:adsk.eagle:package:8700970/2"/>
@@
 <part name="J2" library="sirin-clone-library" library_urn="urn:adsk.eagle:library:9336050" deviceset="USB_MICRO-B" device="" package3d_urn="urn:adsk.eagle:package:10018607/2"/>
 <part name="GND8" library="moon-germs-v1_main" library_urn="urn:adsk.eagle:library:8442267" deviceset="GND" device=""/>
+<part name="U$2" library="sirin-clone-library" library_urn="urn:adsk.eagle:library:9336050" deviceset="TEST_POINT" device="" package3d_urn="urn:adsk.eagle:package:12955547/1"/>
 </parts>
 <sheets>
@@
 <attribute name="VALUE" x="-355.6" y="220.726" size="1.778" layer="96" align="top-center"/>
 </instance>
+<instance part="U$2" gate="G$1" x="-342.9" y="238.76" smashed="yes"/>
 </instances>
 <busses>
@@
 <wire x1="-48.26" y1="57.15" x2="-53.34" y2="57.15" width="0.1524" layer="91"/>
 <wire x1="-53.34" y1="57.15" x2="-53.34" y2="58.42" width="0.1524" layer="91"/>
+<junction x="-53.34" y="57.15"/>
 </segment>
 <segment>
@@
 <wire x1="-350.52" y1="238.76" x2="-358.14" y2="238.76" width="0.1524" layer="91"/>
 <pinref part="J2" gate="J1" pin="VBUS"/>
+<pinref part="U$2" gate="G$1" pin="P$1"/>
+<wire x1="-350.52" y1="238.76" x2="-342.9" y2="238.76" width="0.1524" layer="91"/>
+<junction x="-350.52" y="238.76"/>
 </segment>
 </net>
@@
 </sheet>
 </sheets>
+<errors>
+</errors>
 </schematic>
 </drawing>
