File: hardware/electronics/KELPIE_LOGIC_PCB.sch (EAGLE design)
At the start: 56 parts, among them J1 PJ-002A, J3 30_PIN_CONNECTOR_MALEFLEX_CON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, J5 SWITCHCRAFT_PHONEJACK, J6 SWD_CONNECTOR, T2 MCP1825S, U4 SGTL5000_32QFN, U5 23LC1024

Commit message: update readme
Parts:
- C11, C12: device moon-germs-v1_main:22PF -> sirin-clone-library:22PF
- D5: device moon-germs-v1_main:LED_ORANGE0805 -> sirin-clone-library:LED_ORANGE0805
- D6: device moon-germs-v1_main:AP7313 -> sirin-clone-library:AP7313
- L3: device moon-germs-v1_main:FERRITE600_AUDIO -> sirin-clone-library:FERRITE600_AUDIO
- R5, R6: device moon-germs-v1_main:33OHM -> sirin-clone-library:33OHM
- R7, R8: device moon-germs-v1_main:470OHM -> sirin-clone-library:470OHM
- U$6: device moon-germs-v1_main:MICROSD -> sirin-clone-library:MICROSD
- U4: device moon-germs-v1_main:SGTL5000_32QFN -> sirin-clone-library:SGTL5000_32QFN
- U5: device moon-germs-v1_main:23LC1024 -> sirin-clone-library:23LC1024
Changed lines of the file:
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@@
 </layers>
 <schematic xreflabel="%F%N/%S.%C%R" xrefpart="/%S.%C%R">
+<fusionteam huburn="a.cGVyc29uYWw6dWUyOWViOTli" projecturn="a.cGVyc29uYWw6dWUyOWViOTliIzIwMTkwMjI4MTc5MjYyNDAx" folderUrn="urn:adsk.wipprod:fs.folder:co.8dNkGeL_QFqK5y_dgGXRbQ" urn="urn:adsk.wipprod:dm.lineage:QgZpCW-WRcCZpYZAvfiirQ"  versionUrn="urn:adsk.wipprod:fs.file:vf.QgZpCW-WRcCZpYZAvfiirQ?version=1" camFileUrn="" camFileVersionUrn="" lastpublishedchangeguid="415e3ca6-8c7f-efed-292d-886c2249df73"/>
 <attributes>
 </attributes>
@@
 <part name="C7" library="sirin-clone-library" library_urn="urn:adsk.eagle:library:9336050" deviceset="2.2UF" device="" package3d_urn="urn:adsk.eagle:package:8442351/2"/>
 <part name="GND7" library="moon-germs-v1_main" library_urn="urn:adsk.eagle:library:8442267" deviceset="GND" device=""/>
-<part name="R5" library="moon-germs-v1_main" library_urn="urn:adsk.eagle:library:8442267" deviceset="33OHM" device="" package3d_urn="urn:adsk.eagle:package:8442354/2" value="33"/>
-<part name="R6" library="moon-germs-v1_main" library_urn="urn:adsk.eagle:library:8442267" deviceset="33OHM" device="" package3d_urn="urn:adsk.eagle:package:8442354/2" value="33"/>
+<part name="R5" library="sirin-clone-library" library_urn="urn:adsk.eagle:library:9336050" deviceset="33OHM" device="" package3d_urn="urn:adsk.eagle:package:8442354/2" value="33"/>
+<part name="R6" library="sirin-clone-library" library_urn="urn:adsk.eagle:library:9336050" deviceset="33OHM" device="" package3d_urn="urn:adsk.eagle:package:8442354/2" value="33"/>
 <part name="J6" library="moon-germs-v1_main" library_urn="urn:adsk.eagle:library:8442267" deviceset="SWD_CONNECTOR" device="" package3d_urn="urn:adsk.eagle:package:8709581/1"/>
 <part name="GND9" library="moon-germs-v1_main" library_urn="urn:adsk.eagle:library:8442267" deviceset="GND" device=""/>
@@
 <part name="C10" library="sirin-clone-library" library_urn="urn:adsk.eagle:library:9336050" deviceset="0.1UF" device="" package3d_urn="urn:adsk.eagle:package:8442351/2"/>
 <part name="GND13" library="moon-germs-v1_main" library_urn="urn:adsk.eagle:library:8442267" deviceset="GND" device=""/>
-<part name="R7" library="moon-germs-v1_main" library_urn="urn:adsk.eagle:library:8442267" deviceset="470OHM" device="" package3d_urn="urn:adsk.eagle:package:8442354/2" value="470"/>
-<part name="D5" library="moon-germs-v1_main" library_urn="urn:adsk.eagle:library:8442267" deviceset="LED_ORANGE" device="0805" package3d_urn="urn:adsk.eagle:package:8442343/2" value="ORANGE"/>
+<part name="R7" library="sirin-clone-library" library_urn="urn:adsk.eagle:library:9336050" deviceset="470OHM" device="" package3d_urn="urn:adsk.eagle:package:8442354/2" value="470"/>
+<part name="D5" library="sirin-clone-library" library_urn="urn:adsk.eagle:library:9336050" deviceset="LED_ORANGE" device="0805" package3d_urn="urn:adsk.eagle:package:8442343/2" value="ORANGE"/>
 <part name="GND14" library="moon-germs-v1_main" library_urn="urn:adsk.eagle:library:8442267" deviceset="GND" device=""/>
-<part name="C11" library="moon-germs-v1_main" library_urn="urn:adsk.eagle:library:8442267" deviceset="22PF" device="" package3d_urn="urn:adsk.eagle:package:8442351/2" value="22PF"/>
-<part name="C12" library="moon-germs-v1_main" library_urn="urn:adsk.eagle:library:8442267" deviceset="22PF" device="" package3d_urn="urn:adsk.eagle:package:8442351/2" value="22PF"/>
+<part name="C11" library="sirin-clone-library" library_urn="urn:adsk.eagle:library:9336050" deviceset="22PF" device="" package3d_urn="urn:adsk.eagle:package:8442351/2" value="22PF"/>
+<part name="C12" library="sirin-clone-library" library_urn="urn:adsk.eagle:library:9336050" deviceset="22PF" device="" package3d_urn="urn:adsk.eagle:package:8442351/2" value="22PF"/>
 <part name="GND15" library="moon-germs-v1_main" library_urn="urn:adsk.eagle:library:8442267" deviceset="GND" device=""/>
 <part name="GND16" library="moon-germs-v1_main" library_urn="urn:adsk.eagle:library:8442267" deviceset="GND" device=""/>
 <part name="L1" library="moon-germs-v1_main" library_urn="urn:adsk.eagle:library:8442267" deviceset="FERRITE600_TEENSY" device="" package3d_urn="urn:adsk.eagle:package:8700966/1"/>
-<part name="R8" library="moon-germs-v1_main" library_urn="urn:adsk.eagle:library:8442267" deviceset="470OHM" device="" package3d_urn="urn:adsk.eagle:package:8442354/2" value="470"/>
+<part name="R8" library="sirin-clone-library" library_urn="urn:adsk.eagle:library:9336050" deviceset="470OHM" device="" package3d_urn="urn:adsk.eagle:package:8442354/2" value="470"/>
 <part name="C13" library="sirin-clone-library" library_urn="urn:adsk.eagle:library:9336050" deviceset="2.2UF" device="" package3d_urn="urn:adsk.eagle:package:8442351/2"/>
 <part name="L4" library="moon-germs-v1_main" library_urn="urn:adsk.eagle:library:8442267" deviceset="FERRITE600_TEENSY" device="" package3d_urn="urn:adsk.eagle:package:8700966/1"/>
@@
 <part name="C35" library="sirin-clone-library" library_urn="urn:adsk.eagle:library:9336050" deviceset="0.1UF" device="" package3d_urn="urn:adsk.eagle:package:8442351/2"/>
 <part name="C36" library="sirin-clone-library" library_urn="urn:adsk.eagle:library:9336050" deviceset="0.15UF" device="" package3d_urn="urn:adsk.eagle:package:8442351/2"/>
-<part name="D6" library="moon-germs-v1_main" library_urn="urn:adsk.eagle:library:8442267" deviceset="AP7313" device="" package3d_urn="urn:adsk.eagle:package:8442353/2"/>
-<part name="L3" library="moon-germs-v1_main" library_urn="urn:adsk.eagle:library:8442267" deviceset="FERRITE600_AUDIO" device="" package3d_urn="urn:adsk.eagle:package:8442354/2" value="FER600"/>
+<part name="D6" library="sirin-clone-library" library_urn="urn:adsk.eagle:library:9336050" deviceset="AP7313" device="" package3d_urn="urn:adsk.eagle:package:8442353/2"/>
+<part name="L3" library="sirin-clone-library" library_urn="urn:adsk.eagle:library:9336050" deviceset="FERRITE600_AUDIO" device="" package3d_urn="urn:adsk.eagle:package:8442354/2" value="FER600"/>
 <part name="R11" library="sirin-clone-library" library_urn="urn:adsk.eagle:library:9336050" deviceset="2.2KOHM" device="" package3d_urn="urn:adsk.eagle:package:8442354/2" value="2.2K"/>
 <part name="R12" library="sirin-clone-library" library_urn="urn:adsk.eagle:library:9336050" deviceset="2.2KOHM" device="" package3d_urn="urn:adsk.eagle:package:8442354/2" value="2.2K"/>
-<part name="U4" library="moon-germs-v1_main" library_urn="urn:adsk.eagle:library:8442267" deviceset="SGTL5000_32QFN" device="" package3d_urn="urn:adsk.eagle:package:8442355/2"/>
-<part name="U5" library="moon-germs-v1_main" library_urn="urn:adsk.eagle:library:8442267" deviceset="23LC1024" device="" package3d_urn="urn:adsk.eagle:package:8442350/2"/>
-<part name="U$6" library="moon-germs-v1_main" library_urn="urn:adsk.eagle:library:8442267" deviceset="MICROSD" device="" package3d_urn="urn:adsk.eagle:package:8442348/2"/>
+<part name="U4" library="sirin-clone-library" library_urn="urn:adsk.eagle:library:9336050" deviceset="SGTL5000_32QFN" device="" package3d_urn="urn:adsk.eagle:package:8442355/2"/>
+<part name="U5" library="sirin-clone-library" library_urn="urn:adsk.eagle:library:9336050" deviceset="23LC1024" device="" package3d_urn="urn:adsk.eagle:package:8442350/2"/>
+<part name="U$6" library="sirin-clone-library" library_urn="urn:adsk.eagle:library:9336050" deviceset="MICROSD" device="" package3d_urn="urn:adsk.eagle:package:8442348/2"/>
 <part name="R13" library="sirin-clone-library" library_urn="urn:adsk.eagle:library:9336050" deviceset="10KOHM" device="" package3d_urn="urn:adsk.eagle:package:8442354/2" value="10K"/>
 <part name="R14" library="sirin-clone-library" library_urn="urn:adsk.eagle:library:9336050" deviceset="10KOHM" device="" package3d_urn="urn:adsk.eagle:package:8442354/2" value="10K"/>

Commit message: hardware fix, updated AP7313 regulator from 3.3V to 1.8V reg, thanks @jawsper for catching this
Connections:
- net N$20 renamed 1.8V
Changed lines of the file:
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@@
 </segment>
 </net>
-<net name="N$20" class="0">
+<net name="1.8V" class="0">
 <segment>
 <wire x1="52.07" y1="337.82" x2="54.61" y2="337.82" width="0.1524" layer="91"/>
